Commit message: feat: replaced edrone model with newer swift drone model

File: rotors_description/urdf/component_snippets.xacro (robot description, xacro)
@@ -755,5 +755,5 @@
       measurement_delay="0"
       measurement_divisor="1"
-      mass_imu_sensor="0.015"
+      mass_imu_sensor="0.01"
       gyroscope_noise_density="0.0003394"
       gyroscope_random_walk="0.000038785"
@@ -764,5 +764,5 @@
       accelerometer_bias_correlation_time="300.0"
       accelerometer_turn_on_bias_sigma="0.1960">
-      <inertia ixx="0.00001" ixy="0.0" ixz="0.0" iyy="0.00001" iyz="0.0" izz="0.00001" />
+      <inertia ixx="1.667e-7" ixy="0.0" ixz="0.0" iyy="1.667e-7" iyz="0.0" izz="1.667e-7" />
       <origin xyz="0.015 0 0.0113" rpy="0 0 0" />
     </xacro:imu_plugin_macro>
@@ -777,5 +777,5 @@
       measurement_delay="0"
       measurement_divisor="1"
-      mass_imu_sensor="0.001"
+      mass_imu_sensor="0.01"
       gyroscope_noise_density="0.0"
       gyroscope_random_walk="0.0"
@@ -786,5 +786,5 @@
       accelerometer_bias_correlation_time="300.0"
       accelerometer_turn_on_bias_sigma="0.0">
-      <inertia ixx="0.00001" ixy="0.0" ixz="0.0" iyy="0.00001" iyz="0.0" izz="0.00001" />
+      <inertia ixx="1.667e-7" ixy="0.0" ixz="0.0" iyy="1.667e-7" iyz="0.0" izz="1.667e-7" />
       <origin xyz="0 0 0" rpy="0 0 0" />
     </xacro:imu_plugin_macro>
@@ -801,5 +801,5 @@
       parent_frame_id="world"
       child_frame_id="${namespace}/base_link"
-      mass_odometry_sensor="0.001"
+      mass_odometry_sensor="0.01"
       measurement_divisor="1"
       measurement_delay="0"
@@ -816,5 +816,5 @@
       odometry_map=""
       image_scale="">
-      <inertia ixx="0.00001" ixy="0.0" ixz="0.0" iyy="0.00001" iyz="0.0" izz="0.00001" /> <!-- [kg m^2] [kg m^2] [kg m^2] [kg m^2] [kg m^2] [kg m^2] -->
+      <inertia ixx="1.667e-7" ixy="0.0" ixz="0.0" iyy="1.667e-7" iyz="0.0" izz="1.667e-7" /> <!-- [kg m^2] [kg m^2] [kg m^2] [kg m^2] [kg m^2] [kg m^2] -->
       <origin xyz="0.0 0.0 0.0" rpy="0.0 0.0 0.0" />
     </xacro:odometry_plugin_macro>
@@ -829,5 +829,5 @@
       measurement_delay="0"
       measurement_divisor="1"
-      mass_imu_sensor="0.001"
+      mass_imu_sensor="0.01"
       gyroscope_noise_density="0.0003394"
       gyroscope_random_walk="0.000038785"
@@ -838,5 +838,5 @@
       accelerometer_bias_correlation_time="300.0"
       accelerometer_turn_on_bias_sigma="0.1960">
-      <inertia ixx="0.00001" ixy="0.0" ixz="0.0" iyy="0.00001" iyz="0.0" izz="0.00001" />
+      <inertia ixx="1.667e-7" ixy="0.0" ixz="0.0" iyy="1.667e-7" iyz="0.0" izz="1.667e-7" />
       <origin xyz="0 0 0" rpy="0 0 0" />
     </xacro:imu_plugin_macro>
@@ -854,5 +854,5 @@
         parent_frame_id="world"
         child_frame_id="${namespace}/base_link"
-        mass_odometry_sensor="0.00001"
+        mass_odometry_sensor="0.01"
         measurement_divisor="10"
         measurement_delay="0"
@@ -869,5 +869,5 @@
         odometry_map=""
         image_scale="">
-        <inertia ixx="0.00001" ixy="0.0" ixz="0.0" iyy="0.00001" iyz="0.0" izz="0.00001" /> <!-- [kg m^2] [kg m^2] [kg m^2] [kg m^2] [kg m^2] [kg m^2] -->
+        <inertia ixx="1.667e-7" ixy="0.0" ixz="0.0" iyy="1.667e-7" iyz="0.0" izz="1.667e-7" /> <!-- [kg m^2] [kg m^2] [kg m^2] [kg m^2] [kg m^2] [kg m^2] -->
         <origin xyz="0.0 0.0 0.0" rpy="0.0 0.0 0.0" />
       </xacro:odometry_plugin_macro>
@@ -885,5 +885,5 @@
         parent_frame_id="world"
         child_frame_id="${namespace}/base_link"
-        mass_odometry_sensor="0.00001"
+        mass_odometry_sensor="0.01"
         measurement_divisor="10"
         measurement_delay="0"
@@ -900,5 +900,5 @@
         odometry_map=""
         image_scale="">
-        <inertia ixx="0.00001" ixy="0.0" ixz="0.0" iyy="0.00001" iyz="0.0" izz="0.00001" /> <!-- [kg m^2] [kg m^2] [kg m^2] [kg m^2] [kg m^2] [kg m^2] -->
+        <inertia ixx="1.667e-7" ixy="0.0" ixz="0.0" iyy="1.667e-7" iyz="0.0" izz="1.667e-7" /> <!-- [kg m^2] [kg m^2] [kg m^2] [kg m^2] [kg m^2] [kg m^2] -->
         <origin xyz="0.0 0.0 0.0" rpy="0.0 0.0 0.0" />
       </xacro:odometry_plugin_macro>
@@ -913,5 +913,5 @@
       measurement_delay="0"
       measurement_divisor="1"
-      mass_imu_sensor="0.00001"
+      mass_imu_sensor="0.01"
       gyroscope_noise_density="0.000175"
       gyroscope_random_walk="0.0105"
@@ -922,5 +922,5 @@
       accelerometer_bias_correlation_time="300.0"
       accelerometer_turn_on_bias_sigma="0.588">
-      <inertia ixx="0.00001" ixy="0.0" ixz="0.0" iyy="0.00001" iyz="0.0" izz="0.00001" />
+      <inertia ixx="1.667e-7" ixy="0.0" ixz="0.0" iyy="1.667e-7" iyz="0.0" izz="1.667e-7" />
       <origin xyz="0 0 0" rpy="0 0 0" />
     </xacro:imu_plugin_macro>

File: rotors_description/urdf/multirotor_base.xacro (robot description, xacro)
@@ -36,5 +36,5 @@
 			<link name="${robot_namespace}/base_link"></link>
 			<joint name="${robot_namespace}/base_joint" type="fixed">
-				<origin xyz="0 0 0" rpy="0 0 0" />
+				<origin xyz="0 0 0.04" rpy="0 0 3.1415926" />
 				<parent link="${robot_namespace}/base_link" />
 				<child link="${robot_namespace}/base_link_inertia" />
@@ -50,5 +50,5 @@
 					<geometry>
 						<xacro:if value="${use_mesh_file}">
-							<mesh filename="${mesh_file}" scale="1 1 1" />
+							<mesh filename="${mesh_file}" scale="0.001 0.001 0.001" />
 						</xacro:if>
 						<xacro:unless value="${use_mesh_file}">
@@ -101,5 +101,5 @@
 						<xacro:unless value="${use_own_mesh}">
 							<mesh filename="package://rotors_description/meshes/propeller_${direction}.dae"
-								scale="${radius_rotor} ${radius_rotor} ${radius_rotor}" /> <!-- The propeller meshes have a radius of 1m -->
+								scale="0.001 0.001 0.001" /> <!-- The propeller meshes have a radius of 1m -->
 								<!-- <box size="${2*radius_rotor} 0.01 0.005"/> -->
 							</xacro:unless>
@@ -145,10 +145,4 @@
 				</joint>
 				<link name="${robot_namespace}/motor_${motor_number}">
-					<visual>
-						<geometry>
-					<mesh filename="package://rotors_description/meshes/swift_motor.stl"
-scale="0.002769 0.002769 0.002769" />
-</geometry>
-</visual>
 </link>
 </xacro:macro>

File: rotors_description/urdf/swift.xacro (robot description, xacro)
@@ -6,18 +6,18 @@
   <xacro:property name="use_mesh_file" value="true" />
   <xacro:property name="mesh_file" value="package://rotors_description/meshes/swift_frame.stl" />
-  <xacro:property name="mass" value="1.5" /> <!-- [kg] -->
-  <xacro:property name="body_width" value="0.3" /> <!-- [m] -->
-  <xacro:property name="body_height" value="0.16" /> <!-- [m] -->
-  <xacro:property name="mass_rotor" value="0.005" /> <!-- [kg] -->
-  <xacro:property name="arm_length" value="0.09" /> <!-- [m] -->
+  <xacro:property name="mass" value="0.185" /> <!-- [kg] -->
+  <xacro:property name="body_width" value="0.11" /> <!-- [m] -->
+  <xacro:property name="body_height" value="0.018" /> <!-- [m] -->
+  <xacro:property name="mass_rotor" value="0.0063" /> <!-- [kg] -->
+  <xacro:property name="arm_length" value="0.0345" /> <!-- [m] -->
   <!-- changed from 0.023 to 0.027 -->
-  <xacro:property name="rotor_offset_top" value="0.023" /> <!-- [m] -->
-  <xacro:property name="radius_rotor" value="0.1" /> <!-- [m] -->
-  <xacro:property name="motor_constant" value="8.54858e-06" /> <!-- [kg.m/s^2] -->
-  <xacro:property name="moment_constant" value="0.016" /> <!-- [m] -->
+  <xacro:property name="rotor_offset_top" value="0.053" /> <!-- [m] -->
+  <xacro:property name="radius_rotor" value="0.03175" /> <!-- [m] -->
+  <xacro:property name="motor_constant" value="1.15432e-06" /> <!-- [kg.m/s^2] -->
+  <xacro:property name="moment_constant" value="0.00197" /> <!-- [m] -->
   <xacro:property name="time_constant_up" value="0.0125" /> <!-- [s] -->
   <xacro:property name="time_constant_down" value="0.025" /> <!-- [s] -->
   <xacro:property name="max_rot_velocity" value="838" /> <!-- [rad/s] -->
-    <xacro:property name="motor_offset_top" value="-0.055" />
+  <xacro:property name="motor_offset_top" value="0.038" />
   <xacro:property name="sin30" value="0.5" />
   <xacro:property name="cos30" value="0.866025403784" />
@@ -27,9 +27,9 @@
   <!-- Property Blocks -->
   <xacro:property name="body_inertia">
-    <inertia ixx="0.0347563" ixy="0.0" ixz="0.0" iyy="0.0458929" iyz="0.0" izz="0.0977" /> <!-- [kg.m^2] [kg.m^2] [kg.m^2] [kg.m^2] [kg.m^2] [kg.m^2] -->
+    <xacro:box_inertia x="${body_width}" y="${body_width}" z="${body_height}" mass="${mass}" /> <!-- [kg.m^2] [kg.m^2] [kg.m^2] [kg.m^2] [kg.m^2] [kg.m^2] -->
   </xacro:property>
   <!-- inertia of a single rotor, assuming it is a cuboid. Height=3mm, width=15mm -->
   <xacro:property name="rotor_inertia">
-    <xacro:box_inertia x="${radius_rotor}" y="0.015" z="0.003" mass="${mass_rotor*rotor_velocity_slowdown_sim}" />
+    <xacro:box_inertia x="0.016" y="0.016" z="0.0025" mass="${mass_rotor*rotor_velocity_slowdown_sim}" />
   </xacro:property>
   <!-- Included URDF Files -->
@@ -74,5 +74,5 @@
     robot_namespace="${namespace}"
     suffix="front_right">
-    <origin xyz="${sqrt2 * arm_length} -${sqrt2 * arm_length} ${motor_offset_top}" rpy="1.570796327 0 0"/>
+    <origin xyz="${sqrt2 * arm_length} -${sqrt2 * arm_length} ${motor_offset_top}" rpy="1.57 0 0"/>
   </xacro:vertical_motor>
   <xacro:vertical_rotor
@@ -91,5 +91,5 @@
     rotor_drag_coefficient="${rotor_drag_coefficient}"
     rolling_moment_coefficient="${rolling_moment_coefficient}"
-    color="Blue"
+    color="Orange"
     use_own_mesh="false"
     mesh="">
@@ -103,5 +103,5 @@
     robot_namespace="${namespace}"
     suffix="back_left">
-    <origin xyz="-${sqrt2 * arm_length} ${sqrt2 * arm_length} ${motor_offset_top}" rpy="1.570796327 0 0"/>
+    <origin xyz="-${sqrt2 * arm_length} ${sqrt2 * arm_length} ${motor_offset_top}" rpy="1.57 0 0"/>
   </xacro:vertical_motor>
   <xacro:vertical_rotor robot_namespace="${namespace}"
@@ -119,5 +119,5 @@
     rotor_drag_coefficient="${rotor_drag_coefficient}"
     rolling_moment_coefficient="${rolling_moment_coefficient}"
-    color="Red"
+    color="Green"
     use_own_mesh="false"
     mesh="">
@@ -131,5 +131,5 @@
     robot_namespace="${namespace}"
     suffix="front_left">
-    <origin xyz="${sqrt2 * arm_length} ${sqrt2 * arm_length} ${motor_offset_top}" rpy="1.570796327 0 0"/>
+    <origin xyz="${sqrt2 * arm_length} ${sqrt2 * arm_length} ${motor_offset_top}" rpy="1.57 0 0"/>
   </xacro:vertical_motor>
   <xacro:vertical_rotor robot_namespace="${namespace}"
@@ -147,5 +147,5 @@
     rotor_drag_coefficient="${rotor_drag_coefficient}"
     rolling_moment_coefficient="${rolling_moment_coefficient}"
-    color="Blue"
+    color="Black"
     use_own_mesh="false"
     mesh="">
@@ -159,5 +159,5 @@
     robot_namespace="${namespace}"
     suffix="back_right">
-    <origin xyz="-${sqrt2 * arm_length} -${sqrt2 * arm_length} ${motor_offset_top}" rpy="1.570796327 0 0"/>
+    <origin xyz="-${sqrt2 * arm_length} -${sqrt2 * arm_length} ${motor_offset_top}" rpy="1.57 0 0"/>
   </xacro:vertical_motor>
 </robot>

File: rotors_description/urdf/swift_base.xacro (robot description, xacro)
@@ -4,5 +4,5 @@
   <!-- Instantiate swift_big "mechanics" -->
   <xacro:include filename="$(find rotors_description)/urdf/swift.xacro" />
-  <xacro:include filename="$(find rotors_description)/urdf/whycon_marker_file.xacro"/>
+    <xacro:include filename="$(find rotors_description)/urdf/whycon_marker_file.xacro"/>
   <!-- Instantiate a controller. -->
   <xacro:controller_plugin_macro namespace="${namespace}" imu_sub_topic="imu" />
@@ -14,8 +14,8 @@
   <xacro:default_imu namespace="${namespace}" parent_link="${namespace}/base_link" />
   <xacro:camera_macro namespace="${namespace}" parent_link="${namespace}/base_link" camera_suffix="rgb" frame_rate="30"
-      horizontal_fov="0.872665" image_width="640" image_height="480" image_format="R8G8B8" min_distance="0.1"
+      horizontal_fov="0.872665" image_width="1280" image_height="1280" image_format="R8G8B8" min_distance="0.1"
       max_distance="5" noise_mean="0" noise_stddev="0" enable_visual="false">
-        <box size="0.01 0.01 0.01"/>
-      <origin xyz="0 0 0" rpy="0 1.57 0"/>
+        <box size="0.001 0.05 0.1"/>
+      <origin xyz="0.037 0 0.02" rpy="0 1.570796327 0"/>
     </xacro:camera_macro>
   <xacro:if value="$(arg enable_ground_truth)">

File: rotors_description/urdf/whycon_marker_file.xacro (robot description, xacro)
@@ -20,5 +20,5 @@
 	<xacro:macro name="whycon_marker" params="namespace marker_width marker_radius marker">
 		<joint name="${marker}_joint" type="fixed">
-			<origin xyz="0 0 0.041" rpy="0 0 0"/>
+			<origin xyz="0.04 0 0.06" rpy="0 0 0"/>
 			<parent link="${namespace}/base_link"/>
 			<child link="${marker}_link"/>
@@ -26,7 +26,7 @@
 		<link name="${marker}_link">
 				<visual name='Whycon_Marker'>
-					<origin xyz="-.063 0 0" rpy="0 1.570796327 0"/>
+					<origin xyz="-.043 0 0.0005" rpy="0 0 0"/>
 					<geometry>
-						<mesh filename="package://rotors_description/models/whycon_marker/meshes/whycon_marker.dae" scale="0.25 0.25 0.25"/>
+						<mesh filename="package://rotors_description/models/whycon_marker/meshes/whycon_marker.dae"/>
 					</geometry>
 				</visual>
